File: linear_window_controller.kicad_sch (KiCad schematic)
At the start: 170 parts, among them J1 Motor 2, J10 DCDC_IN, J11 VBus, J12 VCC, J13 GND, J14 PANEL_BTN, J2 Motor 1, J3 Motor 4, J4 Motor 3, J5 Amphenol 10053363-200LF, J6 ATX-24 (Molex 39-28-1243), J7 Link-PP_LPJ0135GDNL, J8 PANEL_LED, J9 Control, P1 ESP32 USB, P2 CONSOLE, Q1 BC817-40(SOT23), Q2 BC817-40(SOT23), Q3 BSS138, Q4 BSS138, SW1 PGM, SW2 Service, SW3 Service, SW4 Service, SW5 Service, SW7 Service, U1 TSOP384xx, U10 TMP112AIDRLR, U11 CP2102N-A01-GQFN24, U12 93LC46BT-E/OT, U13 DM9051, U2 DRV8874, U3 DRV8874, U4 DRV8874, U5 DRV8874, U6 PCF8574APWRG4, U7 LIS3DH, U8 ESP32-S3-WROOM-1-N16R2, U9 TPS562200, Y1 25MHz YXC X322525MOB4SI

Commit message: Change ethernet jack to the (much) more common Hanrun HR911105A (in stead of what was still in my bench drawer) Add smoothing caps on potentiometer output Add separate voltage regulation for the potentiometer vcc Change resistor values of LEDs to be less blindening :]
Parts:
- added C48, C49, C50, C51: 10n, Capacitor_SMD:C_0603_1608Metric, symbol Device:C
- added C52, C53, C54, C55, C56, C57: 1u, Capacitor_SMD:C_0603_1608Metric, symbol Device:C
- added J15: RJ45_Hanrun_HR911105A_Horizontal, Connector_RJ:RJ45_Hanrun_HR911105A_Horizontal, symbol Connector:RJ45_Hanrun_HR911105A_Horizontal
- added JP7: ATX_VSB_OUT, Jumper:SolderJumper-2_P1.3mm_Open_TrianglePad1.0x1.5mm, symbol Jumper:SolderJumper_2_Open
- added JP8: PSMB_ADDR, Jumper:SolderJumper-2_P1.3mm_Open_TrianglePad1.0x1.5mm, symbol Jumper:SolderJumper_2_Open
- added U15: MCP1703Ax-250xxTT, Package_TO_SOT_SMD:SOT-23, symbol Regulator_Linear:MCP1703Ax-250xxTT
- F1: PartNr 01220088Z -> 2x 01220088Z
- J1: Alternative (none) -> Phoenix 1984691; LCSC Part # C5349549 -> C3646874; Manuf MAX -> DORABO; PartCmnt One part for J1/2 -> (none); PartNr MAX MX127S-3.5-10P-GN01-Cu-Y-A -> DB125-3.5-5P-GN-S
- J2: Alternative (none) -> (with J1); LCSC Part # C5349549 -> C3646874; Manuf MAX -> DORABO; PartCmnt One part for J1/2 -> (none); PartNr MAX MX127S-3.5-10P-GN01-Cu-Y-A -> DB125-3.5-5P-GN-S
- J3: Alternative (none) -> Phoenix 1984691; LCSC Part # C5349549 -> C3646874; Manuf MAX -> DORABO; PartCmnt One part for J3/J4 -> (none); PartNr MAX MX127S-3.5-10P-GN01-Cu-Y-A -> DB125-3.5-5P-GN-S
- J4: Alternative (none) -> (with J3); LCSC Part # C5349549 -> C3646874; Manuf MAX -> DORABO; PartCmnt One part for J3/J4 -> (none); PartNr MAX MX127S-3.5-10P-GN01-Cu-Y-A -> DB125-3.5-5P-GN-S
- J5: Alternative (none) -> Amphenol 10053363-200LF
- J9: LCSC Part # C5349547 -> C5443903; Manuf MAX -> Phoenix Contact; PartNr MX127S-3.5-06P-GN01-Cu-Y-A -> 1984659
- R2, R3, R35, R36, R56: value 100 -> 300
- R51, R54: value 300 -> 470
Connections:
- net +3.3V: now also C56.1, U15.3 (VI); no longer J1.5 (Pin_5), J2.5 (Pin_5), J3.5 (Pin_5), J4.5 (Pin_5)
- net +5VSB: now also JP7.1 (A)
- net AVDD: now also J15.4 (TCT), J15.5 (RCT)
- net DCDC_IN: now also JP7.2 (B)
- net DRV1_IPROPI: now also C48.1
- net DRV2_IPROPI: now also C49.1
- net DRV3_IPROPI: now also C50.1
- net DRV4_IPROPI: now also C51.1
- net GND: now also C48.2, C49.2, C50.2, C51.2, C52.2, C53.2, C54.2, C55.2, C56.2, C57.2, J15.8, JP8.2 (B), U15.1 (GND)
- net LAN_ACT: now also J15.10
- net LAN_SPEED: now also J15.11
- net POT1: now also C52.1
- net POT2: now also C53.1
- net POT3: now also C55.1
- net POT4: now also C54.1
- net at J7.1 (RD+), R40.2, U13.3 (RX+): now also J15.3 (RD+)
- net at J7.3 (RD-), R41.2, U13.4 (RX-): now also J15.6 (RD-)
- net at J7.4 (TD+), R42.2, U13.6 (TX+): now also J15.1 (TD+)
- net at J7.6 (TD-), R43.2, U13.7 (TX-): now also J15.2 (TD-)
- net at J5.B27 (ADDR), R27.1: now also JP8.1 (A)
- new net +POT_2.5V: C57.1, J1.5 (Pin_5), J2.5 (Pin_5), J3.5 (Pin_5), J4.5 (Pin_5), U15.2 (VO)
- no-connect marks 24 -> 25
Other:
- moved on the sheet: J1, J2, J3, J4, R16, R21, R26, R9

Commit message: Add channel indication LEDs Add external IO (2 inputs/low power IO, 2 high power OD outputs for e.g. magnetic locks) Swap PCF8574 for PCA9555 16 bit iot expander Add heatsink to board (3D) Add PDF file of V1 schematics
Parts:
- removed U6: PCF8574APWRG4, Package_SO:TSSOP-20_4.4x6.5mm_P0.65mm, symbol Interface_Expansion:PCF8574TS
- added D12: A1, LED_SMD:LED_0603_1608Metric, symbol Device:LED
- added D13: A2, LED_SMD:LED_0603_1608Metric, symbol Device:LED
- added D14: B1, LED_SMD:LED_0603_1608Metric, symbol Device:LED
- added D15: B2, LED_SMD:LED_0603_1608Metric, symbol Device:LED
- added J16: EXT, Connector_PinHeader_2.54mm:PinHeader_1x06_P2.54mm_Vertical, symbol Connector_Generic:Conn_01x06
- added JP9: ADDR, Jumper:SolderJumper-3_P1.3mm_Bridged12_RoundedPad1.0x1.5mm, symbol Jumper:Jumper_3_Bridged12
- added Q5, Q6: Si2318CDS, Package_TO_SOT_SMD:SOT-23, symbol Transistor_FET:Si2319CDS
- added R58, R59, R60, R61: 300, Resistor_SMD:R_0603_1608Metric, symbol Device:R
- added R62, R63: 10k, Resistor_SMD:R_0603_1608Metric, symbol Device:R
- added U17: PCA9555PW, Package_SO:TSSOP-24_4.4x7.8mm_P0.65mm, symbol Interface_Expansion:PCA9555PW
Connections:
- net +3.3V: now also D12.2 (A), D13.2 (A), D14.2 (A), D15.2 (A), JP9.1 (A), U17.24 (VDD)
- net A_DWN: now also U17.17 (IO1_4)
- net A_UP: now also U17.16 (IO1_3)
- net BTN_FUNC: now also U17.15 (IO1_2)
- net B_DWN: now also U17.19 (IO1_6)
- net B_UP: now also U17.18 (IO1_5)
- net GND: now also J16.3 (Pin_3), J16.5 (Pin_5), JP9.3 (B), Q5.2 (S), Q6.2 (S), R62.1, R63.1, U17.12 (VSS), U17.2 (A1), U17.3 (A2)
- net LED_F1: now also U17.13 (IO1_0)
- net LED_F2: now also U17.14 (IO1_1)
- net SCL: now also U17.22 (SCL)
- net SDA: now also U17.23 (SDA)
- net ~{IOEX1_INT}: now also U17.1 (~{INT})
- net ~{nPS_OK}: now also U17.11 (IO0_7)
- new net: D15.1 (K), R61.2
- new net: D13.1 (K), R59.2
- new net: D12.1 (K), R58.2
- new net: D14.1 (K), R60.2
- new net: JP9.2 (C), U17.21 (A0)
- new net EXT_IN1: J16.6 (Pin_6), U17.7 (IO0_3)
- new net EXT_IN2: J16.4 (Pin_4), U17.8 (IO0_4)
- new net EXT_OUT1: Q5.1 (G), R62.2, U17.9 (IO0_5)
- new net EXT_OUT1_OD: J16.2 (Pin_2), Q5.3 (D)
- new net EXT_OUT2: Q6.1 (G), R63.2, U17.10 (IO0_6)
- new net EXT_OUT2_OD: J16.1 (Pin_1), Q6.3 (D)
- new net LED_A1: R58.1, U17.4 (IO0_0)
- new net LED_A2: R59.1, U17.5 (IO0_1)
- new net LED_B1: R60.1, U17.6 (IO0_2)
- new net LED_B2: R61.1, U17.20 (IO1_7)
Other:
- moved on the sheet: C17, D1, D2, DIS1, J14, J8, J9, R2, R3, R35, R36, SW2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
