File: linear_window_controller.kicad_sch (KiCad schematic)
At the start: 198 parts, among them J1 Motor 2, J10 DCDC_IN, J11 VBus, J12 VCC, J13 GND, J14 PANEL_BTN, J15 RJ45_Hanrun_HR911105A_Horizon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, J16 EXT, J2 Motor 1, J3 Motor 4, J4 Motor 3, J5 Amphenol 10053363-200LF, J6 ATX-24 (Molex 39-28-1243), J7 Link-PP_LPJ0135GDNL, J8 PANEL_LED, J9 Control, P1 ESP32 USB, P2 CONSOLE, Q1 BC817-40(SOT23), Q2 BC817-40(SOT23), Q3 BSS138, Q4 BSS138, Q5 Si2318CDS, Q6 Si2318CDS, SW1 PGM, SW2 Service, SW3 Service, SW4 Service, SW5 Service, SW7 Service, U1 TSOP384xx, U10 TMP112AIDRLR, U11 CP2102N-A01-GQFN24, U12 93LC46BT-E/OT, U13 DM9051, U15 MCP1703Ax-250xxTT, U17 PCA9555PW, U2 DRV8874, U3 DRV8874, U4 DRV8874, U5 DRV8874, U7 LIS3DH, U8 ESP32-S3-WROOM-1-N16R2, U9 TPS562200, Y1 25MHz YXC X322525MOB4SI

Commit message: Update PCB to reflect the v2.x update Included PMbus voltage shifter (5V <-> 3.3V)
Parts:
- removed J7: Link-PP_LPJ0135GDNL, iotta_footprints:LinkPP_LPJ0135GDNL, symbol iotta:Link-PP_LPJ0135GDNL
- added D16: EXT1, LED_SMD:LED_0603_1608Metric, symbol Device:LED
- added D17: EXT2, LED_SMD:LED_0603_1608Metric, symbol Device:LED
- added Q7, Q8: BSS138, Package_TO_SOT_SMD:SOT-23, symbol Transistor_FET:BSS138
- added R64, R65: 300, Resistor_SMD:R_0603_1608Metric, symbol Device:R
- J14: value PANEL_BTN -> PANEL BTN
- J16: value EXT -> EXT IO
- J8: value PANEL_LED -> PANEL LED
- renumbered J15 to J7
Connections:
- net +3.3V: now also Q7.1 (G), Q8.1 (G)
- net EXT_OUT1: now also D16.2 (A)
- net EXT_OUT1_OD: now also J16.3 (Pin_3); no longer J16.2 (Pin_2)
- net EXT_OUT2: now also D17.2 (A)
- net EXT_OUT2_OD: now also J16.2 (Pin_2); no longer J16.1 (Pin_1)
- net GND: now also J16.1 (Pin_1), R64.1, R65.1; no longer J16.3 (Pin_3)
- net LED_A1: now also U17.5 (IO0_1); no longer U17.4 (IO0_0)
- net LED_A2: now also U17.4 (IO0_0); no longer U17.5 (IO0_1)
- net PS_SCL: now also Q8.3 (D); no longer JP6.1 (A)
- net PS_SDA: now also Q7.3 (D); no longer JP5.1 (A)
- net at R40.2, U13.3 (RX+): now also J7.1 (TD+); no longer J7.3 (RD+)
- net at R38.1: now also J7.9
- net at R39.1: now also J7.12
- net at R41.2, U13.4 (RX-): now also J7.2 (TD-); no longer J7.6 (RD-)
- net at R42.2, U13.6 (TX+): now also J7.3 (RD+); no longer J7.1 (TD+)
- net at R43.2, U13.7 (TX-): now also J7.6 (RD-); no longer J7.2 (TD-)
- net PS_ON renamed ~{PS_ON}
- new net: JP5.1 (A), Q7.2 (S)
- new net: D16.1 (K), R64.2
- new net: JP6.1 (A), Q8.2 (S)
- new net: D17.1 (K), R65.2
- no-connect marks 25 -> 24
Other:
- note added: "Power"
- note removed: "PSU"
- moved on the sheet: C42, C43, C47, D10, D11, D6, D7, D9, J12, J7, JP5, JP6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
